File: PCBs/Placa_de_energia/placa_de_energia.kicad_pcb (KiCad board)
At the start: 2 copper layers, 36 parts

Commit message: EPS
Parts:
- removed the IN+ at (162.9, 77.4)
- removed the IN+ at (170.9, 72.4)
- added R1: R_Axial_DIN0207_L6.3mm_D2.5mm_P10.16mm_Horizontal, Resistor_THT:R_Axial_DIN0207_L6.3mm_D2.5mm_P10.16mm_Horizontal, F.Cu at (161.5, 79.7)
- added R1: R_Axial_DIN0207_L6.3mm_D2.5mm_P10.16mm_Horizontal, Resistor_THT:R_Axial_DIN0207_L6.3mm_D2.5mm_P10.16mm_Horizontal, F.Cu at (170.1, 72.9)
- moved REF** 7.82 mm to (168.2, 112.1), turned to 180 degrees
- moved REF** 5.45 mm to (161.8, 110.8), turned to -90 degrees
- moved R1 5.29 mm to (171.2, 90.8), turned to 150 degrees
- moved R2 2.32 mm to (168.1, 103.0), turned to 90 degrees
- moved REF** 1.93 mm to (168.0, 129.3), turned to 135 degrees
- moved REF** 1.34 mm to (167.8, 63.7)
Routing:
- net (no net): track 641.0 -> 801.4 mm
Other:
- board text added: "B1"
- board text added: "B2"
- board text added: "T1"
- board text added: "T2"
- board text removed: "A0"
- board text removed: "A1"
- board text removed: "A2"
- board text removed: "A3"
- board text removed: "A6"
- board text removed: "A7"
