File: PCBs/Computador de bordo/Computador de bordo.kicad_pcb (KiCad board)
At the start: 2 copper layers, 29 parts

Commit message: up
Parts:
- removed ?: PinHeader_1x02_P2.54mm_Vertical, Connector_PinHeader_2.54mm:PinHeader_1x02_P2.54mm_Vertical
- removed ?: PinHeader_1x03_P2.54mm_Vertical, Connector_PinHeader_2.54mm:PinHeader_1x03_P2.54mm_Vertical
- removed the REF** at (121.1, 134.2)
- removed the REF** at (114.2, 123.1)
- removed the REF** at (145.5, 120.7)
- removed the REF** at (136.2, 133.2)
- removed the REF** at (103.8, 126.0)
- removed the REF** at (136.2, 123.6)
- removed the REF** at (107.6, 114.9)
- removed the REF** at (123.6, 123.8)
- removed the REF** at (100.3, 93.2)
- removed the REF** at (100.3, 108.4)
- removed the REF** at (143.7, 92.5)
- removed the REF** at (153.1, 91.4)
- removed the REF** at (159.2, 87.4)
- removed the REF** at (164.2, 84.1)
- added REF**: ESP32-DevKitC, Espressif:ESP32-DevKitC, F.Cu at (148.6, 97.2)
- moved REF** 83.9 mm to (201.9, 109.9)
Routing:
- net (no net): track 1769.5 -> 31.0 mm
Other:
- net class Default removed

Commit message: OBDH
Parts:
- removed the REF** at (168.5, 63.3)
- removed the REF** at (201.9, 109.9)
- removed the REF** at (160.4, 62.6)
- removed the REF** at (161.0, 70.7)
- removed the REF** at (165.2, 67.5)
- moved REF** 50.4 mm to (106.0, 84.5), turned to 90 degrees
- moved REF** 11.4 mm to (158.8, 102.2), turned to 180 degrees
Routing:
- net (no net): track 31.0 -> 1085.8 mm, vias 0 -> 1
Other:
- board text added: "12"
- board text added: "14"
- board text added: "25"
- board text added: "26"
- board text added: "27"
- board text added: "32"
- board text added: "33"
- board text added: "34"
- board text added: "35"
- board text added: "36"
- board text added: "39"
- board text added: "OBDH"
- board text added: "RX"
- board text added: "TX"
- board text removed: "0"
- board text removed: "1"
- board text removed: "7"
- board text removed: "8"
- board text removed: "9"
- board text removed: "A0"
- board text removed: "A1"
- board text removed: "A2"
- board text removed: "A3"
- board text removed: "A6"
- board text removed: "A7"
- board text removed: "MISO"
- board text removed: "MOSI"
- board text removed: "SCK"
